Commit message: exported mesh to .obj and read mesh data

File: urdf/quadrotor_base.urdf.xacro (robot description, xacro)
@@ -18,7 +18,7 @@
       </visual>
       <collision>
-        <origin xyz="0 0 0" rpy="0 0 0" />
+        <origin xyz="-1 0.5 0.3" rpy="0 0 0" />
         <geometry>
-          <mesh filename="package://hector_quadrotor_description/meshes/quadrotor/quadrotor_base.stl"/>
+          <mesh filename="package://hector_quadrotor_description/meshes/quadrotor/quadrotor_base.obj"/>
         </geometry>
       </collision>
