Commit message: new drone, clean urdf folder

File: urdf/quadrotor.urdf.xacro (robot description, xacro)
@@ -5,5 +5,5 @@
 >
     <!-- Included URDF Files -->
-    <xacro:include filename="$(find hector_quadrotor_description)/urdf/quadrotor_base.urdf.xacro" />
+    <xacro:include filename="$(find drone_planning)/urdf/quadrotor_base.urdf.xacro" />
     <!-- Instantiate quadrotor_base_macro once (has no parameters atm) -->
     <xacro:quadrotor_base_macro />

File: urdf/quadrotor_base.urdf.xacro (robot description, xacro)
@@ -14,5 +14,5 @@
         <origin xyz="-1 0.5 0.3" rpy="0 0 0" />
         <geometry>
-          <mesh filename="package://hector_quadrotor_description/meshes/quadrotor/quadrotor_base.dae"/>
+          <mesh filename="package://drone_planning/meshes/quadrotor/quadrotor_2.dae"/>
         </geometry>
       </visual>
@@ -20,5 +20,5 @@
         <origin xyz="-1 0.5 0.3" rpy="0 0 0" />
         <geometry>
-          <mesh filename="package://hector_quadrotor_description/meshes/quadrotor/quadrotor_base.obj"/>
+          <mesh filename="package://drone_planning/meshes/quadrotor/quadrotor_2.obj"/>
         </geometry>
       </collision>

Commit message: Change launch and urdf files

File: urdf/quadrotor.urdf.xacro (robot description, xacro)
@@ -4,7 +4,26 @@
   xmlns:xacro="http://ros.org/wiki/xacro"
 >
-    <!-- Included URDF Files -->
-    <xacro:include filename="$(find drone_planning)/urdf/quadrotor_base.urdf.xacro" />
-    <!-- Instantiate quadrotor_base_macro once (has no parameters atm) -->
-    <xacro:quadrotor_base_macro />
+<!--    -->
+<xacro:property name="Xpos" value="-1.0"/>
+<xacro:property name="Ypos" value="0.5"/>
+<xacro:property name="Zpos" value="0.3"/>
+    <link name="odom">
+      <inertial>
+        <mass value="1.477" />
+        <origin xyz="0 0 0" />
+        <inertia ixx="0.01152" ixy="0.0" ixz="0.0" iyy="0.01152" iyz="0.0" izz="0.0218" />
+      </inertial>
+      <visual>
+        <origin xyz="${Xpos} ${Ypos} ${Zpos}" rpy="0 0 0" />
+        <geometry>
+          <mesh filename="package://drone_planning/meshes/quadrotor/quadrotor_2.dae"/>
+        </geometry>
+      </visual>
+      <collision>
+        <origin xyz="${Xpos} ${Ypos} ${Zpos}" rpy="0 0 0" />
+        <geometry>
+          <mesh filename="package://drone_planning/meshes/quadrotor/quadrotor_2.obj"/>
+        </geometry>
+      </collision>
+    </link>
 </robot>

File: urdf/quadrotor_base.urdf.xacro (robot description, xacro)
@@ -1,6 +1,7 @@
 <?xml version="1.0"?>
 <robot xmlns:xacro="http://ros.org/wiki/xacro">
-  <!--<xacro:include filename="$(find hector_sensors_description)/urdf/sonar_sensor.urdf.xacro" />-->
-  <xacro:property name="pi" value="3.1415926535897931" />
+<!--<xacro:property name="Xpos" value="1"/>-->
+<xacro:property name="Ypos" value="0.5"/>
+<xacro:property name="Zpos" value="0.3"/>
   <!-- Main quadrotor link -->
   <xacro:macro name="quadrotor_base_macro">
@@ -12,5 +13,5 @@
       </inertial>
       <visual>
-        <origin xyz="-1 0.5 0.3" rpy="0 0 0" />
+        <origin xyz="${Xpos} ${Ypos} ${Zpos}" rpy="0 0 0" />
         <geometry>
           <mesh filename="package://drone_planning/meshes/quadrotor/quadrotor_2.dae"/>
@@ -18,5 +19,5 @@
       </visual>
       <collision>
-        <origin xyz="-1 0.5 0.3" rpy="0 0 0" />
+        <origin xyz="${Xpos} ${Ypos} ${Zpos}" rpy="0 0 0" />
         <geometry>
           <mesh filename="package://drone_planning/meshes/quadrotor/quadrotor_2.obj"/>
@@ -24,8 +25,4 @@
       </collision>
     </link>
-    <!-- Sonar height sensor -->
-    <!--<xacro:sonar_sensor name="sonar" parent="base_link" ros_topic="sonar_height" update_rate="10" min_range="0.03" max_range="3.0" field_of_view="${40*pi/180}" ray_count="3">
-      <origin xyz="-0.16 0.0 -0.012" rpy="0 ${90*pi/180} 0"/>
-    </xacro:sonar_sensor>-->
   </xacro:macro>
 </robot>

Commit message: Test link added

File: urdf/quadrotor.urdf.xacro (robot description, xacro)
@@ -8,8 +8,16 @@
 <xacro:property name="Ypos" value="0.5"/>
 <xacro:property name="Zpos" value="0.3"/>
-    <link name="odom">
+  <link name="test_link">
+    <visual>
+      <origin xyz="${Xpos} ${Ypos} ${Zpos}" rpy="0 0 0" />
+      <geometry>
+        <cylinder length="0.1" radius="0.1"/>
+      </geometry>
+    </visual>
+  </link>
+  <link name="odom">
       <inertial>
         <mass value="1.477" />
-        <origin xyz="0 0 0" />
+        <origin xyz="0 0 0" rpy="0 0 0" />
         <inertia ixx="0.01152" ixy="0.0" ixz="0.0" iyy="0.01152" iyz="0.0" izz="0.0218" />
       </inertial>
@@ -17,4 +25,5 @@
         <origin xyz="${Xpos} ${Ypos} ${Zpos}" rpy="0 0 0" />
         <geometry>
+          <!--<cylinder length="0.1" radius="0.2"/>-->
           <mesh filename="package://drone_planning/meshes/quadrotor/quadrotor_2.dae"/>
         </geometry>
@@ -27,3 +36,7 @@
       </collision>
     </link>
+  <joint name="test_joint" type="fixed">
+    <parent link="test_link"/>
+    <child link="odom"/>
+  </joint>
 </robot>
